File: cassette.kicad_sch (KiCad schematic)
At the start: 21 parts

Commit message: Implement power transform circuit
Parts:
- C43: renamed from C32; value (none) -> 1uF; footprint (none) -> artemisa:Radial_capacitor
- C44: renamed from C33; value (none) -> 22nF; footprint (none) -> artemisa:Disc_capacitor
- C45: renamed from C?; value (none) -> 100nF; footprint (none) -> artemisa:Disc_capacitor
- C46: renamed from C34; value (none) -> 22nF; footprint (none) -> artemisa:Disc_capacitor
- C47: renamed from C35; value (none) -> 1uF; footprint (none) -> artemisa:Radial_capacitor
- D5: renamed from D3; value (none) -> 1N4448; footprint (none) -> artemisa:Axial_diode
- J7: renamed from J8; value (none) -> DIN8; footprint (none) -> artemisa:DIN8
- K1: value (none) -> Relay; footprint (none) -> artemisa:Relay
- Q2: value (none) -> 2N2907; footprint (none) -> artemisa:TO92
- R15: renamed from R?; value (none) -> 1k; footprint (none) -> artemisa:Axial_resistor
- R16, R18, R20: renamed from R?; value (none) -> 4k7; footprint (none) -> artemisa:Axial_resistor
- R17: renamed from R?; value (none) -> 2k2; footprint (none) -> artemisa:Axial_resistor
- R19: renamed from R?; value (none) -> 100; footprint (none) -> artemisa:Axial_resistor
- R21: renamed from R?; value (none) -> 220k; footprint (none) -> artemisa:Axial_resistor
- R22: renamed from R?; value (none) -> 10k; footprint (none) -> artemisa:Axial_resistor
- R23, R24: renamed from R?; value (none) -> 2k7; footprint (none) -> artemisa:Axial_resistor
- U32: renamed from U19; value (none) -> LM311; footprint (none) -> artemisa:DIP-8_300
- U32: renamed from U?; value (none) -> LM311; footprint (none) -> artemisa:DIP-8_300
Connections:
- net VCC: now reaches R15.2
- net VCC: now also C45.1, D5.2, K1.1, R21.2, R23.2, U32.8 (VCC)
