File: psg.kicad_sch (KiCad schematic)
At the start: 21 parts

Commit message: Implement power transform circuit
Parts:
- C37: renamed from C29; value (none) -> 10u; footprint (none) -> artemisa:Radial_capacitor
- C38: renamed from C30; value (none) -> 10u; footprint (none) -> artemisa:Radial_capacitor
- C39, C41, C42: renamed from C?; value (none) -> 100nF; footprint (none) -> artemisa:Disc_capacitor
- C40: renamed from C31; value (none) -> 10u; footprint (none) -> artemisa:Radial_capacitor
- J5: renamed from J6; value (none) -> CONN_JOY; footprint (none) -> artemisa:Joystick_conn
- J6: renamed from J7; value (none) -> CONN_JOY; footprint (none) -> artemisa:Joystick_conn
- R10: renamed from R?; value (none) -> 4k7; footprint (none) -> artemisa:Axial_resistor
- R11: renamed from R?; value (none) -> 2k7; footprint (none) -> artemisa:Axial_resistor
- R12: renamed from R?; value (none) -> 470; footprint (none) -> artemisa:Axial_resistor
- R13, R14: renamed from R?; value (none) -> 10K; footprint (none) -> artemisa:Axial_resistor
- R9: renamed from R?; value (none) -> 20k; footprint (none) -> artemisa:Axial_resistor
- RN4: value (none) -> 10K; footprint (none) -> artemisa:RN8
- RN5: value (none) -> 10K; footprint (none) -> artemisa:RN4
- U17: renamed from U16; value (none) -> 74LS07; footprint (none) -> artemisa:DIP-14_300
- U29: renamed from U24; value (none) -> AY-3-8910; footprint (none) -> artemisa:DIP-40_600
- U30: renamed from U23; value (none) -> 74HC157; footprint (none) -> artemisa:DIP-16_300
- U31: renamed from U25; value (none) -> 74HC157; footprint (none) -> artemisa:DIP-16_300
- U6: renamed from U14; value (none) -> 74HC08; footprint (none) -> artemisa:DIP-14_300
Connections:
- net VCC: now also C39.1, C41.1, C42.1, J5.5 (VCC), J6.5 (VCC), R14.1, RN4.1, RN5.1, U29.25 (A8), U29.28 (BC2), U29.40 (VCC), U30.16 (VCC), U31.16 (VCC)
