File: ram.kicad_sch (KiCad schematic)
At the start: 4 parts

Commit message: Implement power transform circuit
Parts:
- C34, C35: renamed from C?; value (none) -> 100nF; footprint (none) -> artemisa:Disc_capacitor
- U26: renamed from U1; value (none) -> 62256; footprint (none) -> artemisa:DIP-28_600
- U27: renamed from U2; value (none) -> 62256; footprint (none) -> artemisa:DIP-28_600
Connections:
- net VCC: now reaches C34.1, U26.28 (VCC)
- net VCC: now also C35.1, U27.28 (VCC)
Changed lines of the file:
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@@
   (symbol (lib_id "artemisa:62256") (at 128.27 77.47 0) (unit 1)
     (in_bom yes) (on_board yes)
-    (property "Reference" "U1" (id 0) (at 119.38 55.88 0)
-      (effects (font (size 1.524 1.524)))
-    )
-    (property "Value" "" (id 1) (at 115.57 96.52 0)
-      (effects (font (size 1.524 1.524)))
-    )
-    (property "Footprint" "" (id 2) (at 128.27 81.28 0)
+    (property "Reference" "U26" (id 0) (at 119.38 55.88 0)
+      (effects (font (size 1.524 1.524)))
+    )
+    (property "Value" "62256" (id 1) (at 115.57 96.52 0)
+      (effects (font (size 1.524 1.524)))
+    )
+    (property "Footprint" "artemisa:DIP-28_600" (id 2) (at 128.27 81.28 0)
       (effects (font (size 1.524 1.524)) hide)
     )
@@
   (symbol (lib_id "artemisa:62256") (at 207.01 77.47 0) (unit 1)
     (in_bom yes) (on_board yes)
-    (property "Reference" "U2" (id 0) (at 198.12 55.88 0)
-      (effects (font (size 1.524 1.524)))
-    )
-    (property "Value" "" (id 1) (at 194.31 96.52 0)
-      (effects (font (size 1.524 1.524)))
-    )
-    (property "Footprint" "" (id 2) (at 207.01 81.28 0)
+    (property "Reference" "U27" (id 0) (at 198.12 55.88 0)
+      (effects (font (size 1.524 1.524)))
+    )
+    (property "Value" "62256" (id 1) (at 194.31 96.52 0)
+      (effects (font (size 1.524 1.524)))
+    )
+    (property "Footprint" "artemisa:DIP-28_600" (id 2) (at 207.01 81.28 0)
       (effects (font (size 1.524 1.524)) hide)
     )
@@
   (symbol (lib_id "artemisa:GND") (at 128.27 100.33 0) (unit 1)
     (in_bom yes) (on_board yes)
-    (property "Reference" "#PWR05" (id 0) (at 128.27 102.87 0)
-      (effects (font (size 1.524 1.524)) hide)
-    )
-    (property "Value" "" (id 1) (at 128.27 97.79 0)
+    (property "Reference" "#PWR098" (id 0) (at 128.27 102.87 0)
+      (effects (font (size 1.524 1.524)) hide)
+    )
+    (property "Value" "GND" (id 1) (at 128.27 97.79 0)
       (effects (font (size 1.524 1.524)) hide)
     )
@@
   (symbol (lib_id "artemisa:GND") (at 207.01 100.33 0) (unit 1)
     (in_bom yes) (on_board yes)
-    (property "Reference" "#PWR06" (id 0) (at 207.01 102.87 0)
-      (effects (font (size 1.524 1.524)) hide)
-    )
-    (property "Value" "" (id 1) (at 207.01 97.79 0)
+    (property "Reference" "#PWR0101" (id 0) (at 207.01 102.87 0)
+      (effects (font (size 1.524 1.524)) hide)
+    )
+    (property "Value" "GND" (id 1) (at 207.01 97.79 0)
       (effects (font (size 1.524 1.524)) hide)
     )
@@
   (symbol (lib_id "artemisa:VCC") (at 128.27 44.45 0) (unit 1)
     (in_bom yes) (on_board yes)
-    (property "Reference" "#PWR01" (id 0) (at 128.27 45.72 0)
-      (effects (font (size 1.524 1.524)) hide)
-    )
-    (property "Value" "" (id 1) (at 128.27 38.1 0)
+    (property "Reference" "#PWR097" (id 0) (at 128.27 45.72 0)
+      (effects (font (size 1.524 1.524)) hide)
+    )
+    (property "Value" "VCC" (id 1) (at 128.27 38.1 0)
       (effects (font (size 1.524 1.524)) hide)
     )
@@
       (effects (font (size 1.524 1.524)) hide)
     )
+    (pin "1")
+  )
+  (symbol (lib_id "artemisa:Cap") (at 134.62 48.26 90) (unit 1)
+    (in_bom yes) (on_board yes)
+    (property "Reference" "C34" (id 0) (at 133.35 46.99 90)
+      (effects (font (size 1.27 1.27)) (justify left))
+    )
+    (property "Value" "100nF" (id 1) (at 142.24 46.99 90)
+      (effects (font (size 1.27 1.27)) (justify left))
+    )
+    (property "Footprint" "artemisa:Disc_capacitor" (id 2) (at 134.62 48.26 0)
+      (effects (font (size 1.27 1.27)) hide)
+    )
+    (property "Datasheet" "" (id 3) (at 134.62 48.26 0)
+      (effects (font (size 1.27 1.27)) hide)
+    )
+    (pin "1")
+    (pin "2")
+  )
+  (symbol (lib_id "artemisa:GND") (at 139.7 50.8 0) (unit 1)
+    (in_bom yes) (on_board yes)
+    (property "Reference" "#PWR099" (id 0) (at 139.7 53.34 0)
+      (effects (font (size 1.524 1.524)) hide)
+    )
+    (property "Value" "GND" (id 1) (at 139.7 48.26 0)
+      (effects (font (size 1.524 1.524)) hide)
+    )
+    (property "Footprint" "" (id 2) (at 139.7 50.8 0)
+      (effects (font (size 1.524 1.524)) hide)
+    )
+    (property "Datasheet" "" (id 3) (at 139.7 50.8 0)
+      (effects (font (size 1.524 1.524)) hide)
+    )
     (pin "~")
   )
-  (symbol (lib_id "artemisa:Cap") (at 134.62 48.26 90) (unit 1)
-    (in_bom yes) (on_board yes)
-    (property "Reference" "C?" (id 0) (at 133.35 46.99 90)
-      (effects (font (size 1.27 1.27)) (justify left))
-    )
-    (property "Value" "" (id 1) (at 142.24 46.99 90)
-      (effects (font (size 1.27 1.27)) (justify left))
-    )
-    (property "Footprint" "" (id 2) (at 134.62 48.26 0)
-      (effects (font (size 1.27 1.27)) hide)
-    )
-    (property "Datasheet" "" (id 3) (at 134.62 48.26 0)
-      (effects (font (size 1.27 1.27)) hide)
-    )
-    (pin "1")
-    (pin "2")
-  )
-  (symbol (lib_id "artemisa:GND") (at 139.7 50.8 0) (unit 1)
-    (in_bom yes) (on_board yes)
-    (property "Reference" "#PWR03" (id 0) (at 139.7 53.34 0)
-      (effects (font (size 1.524 1.524)) hide)
-    )
-    (property "Value" "" (id 1) (at 139.7 48.26 0)
-      (effects (font (size 1.524 1.524)) hide)
-    )
-    (property "Footprint" "" (id 2) (at 139.7 50.8 0)
-      (effects (font (size 1.524 1.524)) hide)
-    )
-    (property "Datasheet" "" (id 3) (at 139.7 50.8 0)
-      (effects (font (size 1.524 1.524)) hide)
-    )
-    (pin "~")
-  )
   (symbol (lib_id "artemisa:VCC") (at 207.01 44.45 0) (unit 1)
     (in_bom yes) (on_board yes)
-    (property "Reference" "#PWR02" (id 0) (at 207.01 45.72 0)
-      (effects (font (size 1.524 1.524)) hide)
-    )
-    (property "Value" "" (id 1) (at 207.01 38.1 0)
+    (property "Reference" "#PWR0100" (id 0) (at 207.01 45.72 0)
+      (effects (font (size 1.524 1.524)) hide)
+    )
+    (property "Value" "VCC" (id 1) (at 207.01 38.1 0)
       (effects (font (size 1.524 1.524)) hide)
     )
@@
       (effects (font (size 1.524 1.524)) hide)
     )
-    (pin "~")
+    (pin "1")
   )
   (symbol (lib_id "artemisa:Cap") (at 213.36 48.26 90) (unit 1)
     (in_bom yes) (on_board yes)
-    (property "Reference" "C?" (id 0) (at 212.09 46.99 90)
-      (effects (font (size 1.27 1.27)) (justify left))
-    )
-    (property "Value" "" (id 1) (at 220.98 46.99 90)
-      (effects (font (size 1.27 1.27)) (justify left))
-    )
-    (property "Footprint" "" (id 2) (at 213.36 48.26 0)
+    (property "Reference" "C35" (id 0) (at 212.09 46.99 90)
+      (effects (font (size 1.27 1.27)) (justify left))
+    )
+    (property "Value" "100nF" (id 1) (at 220.98 46.99 90)
+      (effects (font (size 1.27 1.27)) (justify left))
+    )
+    (property "Footprint" "artemisa:Disc_capacitor" (id 2) (at 213.36 48.26 0)
       (effects (font (size 1.27 1.27)) hide)
     )
@@
   (symbol (lib_id "artemisa:GND") (at 218.44 50.8 0) (unit 1)
     (in_bom yes) (on_board yes)
-    (property "Reference" "#PWR04" (id 0) (at 218.44 53.34 0)
-      (effects (font (size 1.524 1.524)) hide)
-    )
-    (property "Value" "" (id 1) (at 218.44 48.26 0)
-      (effects (font (size 1.524 1.524)) hide)
-    )
+    (property "Reference" "#PWR0102" (id 0) (at 218.44 53.34 0)
+      (effects (font (size 1.524 1.524)) hide)
+    )
+    (property "Value" "GND" (id 1) (at 218.44 48.26 0)
+      (effects (font (size 1.524 1.524)) hide)
+    )
