File: rom.kicad_sch (KiCad schematic)
At the start: 7 parts

Commit message: Implement power transform circuit
Parts:
- C33: renamed from C?; value (none) -> 100nF; footprint (none) -> artemisa:Disc_capacitor
- JP1, JP2, JP3, JP4: value (none) -> Jumper; footprint (none) -> artemisa:Jumper
- RN2: renamed from RN1; value (none) -> 10K; footprint (none) -> artemisa:RN4
- U25: renamed from U20; value (none) -> SST39SF0; footprint (none) -> artemisa:DIP-32_600
Connections:
- net VCC: now reaches U25.31 (~{WE})
- net VCC: now also C33.1, JP1.1, JP2.1, JP3.1, JP4.1, U25.32 (VCC)
Changed lines of the file:
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@@
   (symbol (lib_id "artemisa:SST39SF0") (at 139.7 69.85 0) (unit 1)
     (in_bom yes) (on_board yes)
-    (property "Reference" "U20" (id 0) (at 133.35 48.26 0)
+    (property "Reference" "U25" (id 0) (at 133.35 48.26 0)
       (effects (font (size 1.524 1.524)))
     )
-    (property "Value" "" (id 1) (at 147.32 101.6 0)
+    (property "Value" "SST39SF0" (id 1) (at 147.32 101.6 0)
       (effects (font (size 1.524 1.524)))
     )
-    (property "Footprint" "" (id 2) (at 139.7 69.85 0)
+    (property "Footprint" "artemisa:DIP-32_600" (id 2) (at 139.7 69.85 0)
       (effects (font (size 1.524 1.524)) hide)
     )
@@
   (symbol (lib_id "artemisa:VCC") (at 161.29 77.47 0) (unit 1)
     (in_bom yes) (on_board yes)
-    (property "Reference" "#PWR062" (id 0) (at 161.29 78.74 0)
-      (effects (font (size 1.524 1.524)) hide)
-    )
-    (property "Value" "" (id 1) (at 161.29 71.12 0)
+    (property "Reference" "#PWR096" (id 0) (at 161.29 78.74 0)
+      (effects (font (size 1.524 1.524)) hide)
+    )
+    (property "Value" "VCC" (id 1) (at 161.29 71.12 0)
       (effects (font (size 1.524 1.524)) hide)
     )
@@
       (effects (font (size 1.524 1.524)) hide)
     )
-    (pin "~")
+    (pin "1")
   )
   (symbol (lib_id "artemisa:Jumper") (at 110.49 158.75 270) (unit 1)
@@
       (effects (font (size 1.524 1.524)) (justify left))
     )
-    (property "Value" "" (id 1) (at 113.0808 160.0962 90)
-      (effects (font (size 1.524 1.524)) (justify left) hide)
-    )
-    (property "Footprint" "" (id 2) (at 110.49 158.75 0)
+    (property "Value" "Jumper" (id 1) (at 113.0808 160.0962 90)
+      (effects (font (size 1.524 1.524)) (justify left) hide)
+    )
+    (property "Footprint" "artemisa:Jumper" (id 2) (at 110.49 158.75 0)
       (effects (font (size 1.524 1.524)) hide)
     )
@@
       (effects (font (size 1.524 1.524)) (justify left))
     )
-    (property "Value" "" (id 1) (at 120.7008 160.0962 90)
-      (effects (font (size 1.524 1.524)) (justify left) hide)
-    )
-    (property "Footprint" "" (id 2) (at 118.11 158.75 0)
+    (property "Value" "Jumper" (id 1) (at 120.7008 160.0962 90)
+      (effects (font (size 1.524 1.524)) (justify left) hide)
+    )
+    (property "Footprint" "artemisa:Jumper" (id 2) (at 118.11 158.75 0)
       (effects (font (size 1.524 1.524)) hide)
     )
@@
       (effects (font (size 1.524 1.524)) (justify left))
     )
-    (property "Value" "" (id 1) (at 128.3208 160.0962 90)
-      (effects (font (size 1.524 1.524)) (justify left) hide)
-    )
-    (property "Footprint" "" (id 2) (at 125.73 158.75 0)
+    (property "Value" "Jumper" (id 1) (at 128.3208 160.0962 90)
+      (effects (font (size 1.524 1.524)) (justify left) hide)
+    )
+    (property "Footprint" "artemisa:Jumper" (id 2) (at 125.73 158.75 0)
       (effects (font (size 1.524 1.524)) hide)
     )
@@
       (effects (font (size 1.524 1.524)) (justify left))
     )
-    (property "Value" "" (id 1) (at 135.9408 160.0962 90)
-      (effects (font (size 1.524 1.524)) (justify left) hide)
-    )
-    (property "Footprint" "" (id 2) (at 133.35 158.75 0)
+    (property "Value" "Jumper" (id 1) (at 135.9408 160.0962 90)
+      (effects (font (size 1.524 1.524)) (justify left) hide)
+    )
+    (property "Footprint" "artemisa:Jumper" (id 2) (at 133.35 158.75 0)
       (effects (font (size 1.524 1.524)) hide)
     )
@@
   (symbol (lib_id "artemisa:RN4") (at 132.08 133.35 180) (unit 1)
     (in_bom yes) (on_board yes)
-    (property "Reference" "RN1" (id 0) (at 137.668 133.2738 0)
+    (property "Reference" "RN2" (id 0) (at 137.668 133.2738 0)
       (effects (font (size 1.524 1.524)) (justify right))
     )
-    (property "Value" "" (id 1) (at 137.668 135.9662 0)
+    (property "Value" "10K" (id 1) (at 137.668 135.9662 0)
       (effects (font (size 1.524 1.524)) (justify right))
     )
-    (property "Footprint" "" (id 2) (at 129.54 131.445 0)
+    (property "Footprint" "artemisa:RN4" (id 2) (at 129.54 131.445 0)
       (effects (font (size 1.524 1.524)) hide)
     )
@@
   (symbol (lib_id "artemisa:GND") (at 132.08 139.7 0) (unit 1)
     (in_bom yes) (on_board yes)
-    (property "Reference" "#PWR064" (id 0) (at 132.08 142.24 0)
-      (effects (font (size 1.524 1.524)) hide)
-    )
-    (property "Value" "" (id 1) (at 132.08 137.16 0)
+    (property "Reference" "#PWR090" (id 0) (at 132.08 142.24 0)
+      (effects (font (size 1.524 1.524)) hide)
+    )
+    (property "Value" "GND" (id 1) (at 132.08 137.16 0)
       (effects (font (size 1.524 1.524)) hide)
     )
@@
   (symbol (lib_id "artemisa:VCC") (at 146.05 147.32 0) (unit 1)
     (in_bom yes) (on_board yes)
-    (property "Reference" "#PWR065" (id 0) (at 146.05 148.59 0)
-      (effects (font (size 1.524 1.524)) hide)
-    )
-    (property "Value" "" (id 1) (at 146.05 140.97 0)
+    (property "Reference" "#PWR093" (id 0) (at 146.05 148.59 0)
+      (effects (font (size 1.524 1.524)) hide)
+    )
+    (property "Value" "VCC" (id 1) (at 146.05 140.97 0)
       (effects (font (size 1.524 1.524)) hide)
     )
@@
       (effects (font (size 1.524 1.524)) hide)
     )
+    (pin "1")
+  )
+  (symbol (lib_id "artemisa:GND") (at 146.05 170.18 0) (unit 1)
+    (in_bom yes) (on_board yes)
+    (property "Reference" "#PWR094" (id 0) (at 146.05 172.72 0)
+      (effects (font (size 1.524 1.524)) hide)
+    )
+    (property "Value" "GND" (id 1) (at 146.05 167.64 0)
+      (effects (font (size 1.524 1.524)) hide)
+    )
+    (property "Footprint" "" (id 2) (at 146.05 170.18 0)
+      (effects (font (size 1.524 1.524)) hide)
+    )
+    (property "Datasheet" "" (id 3) (at 146.05 170.18 0)
+      (effects (font (size 1.524 1.524)) hide)
+    )
     (pin "~")
   )
-  (symbol (lib_id "artemisa:GND") (at 146.05 170.18 0) (unit 1)
-    (in_bom yes) (on_board yes)
-    (property "Reference" "#PWR066" (id 0) (at 146.05 172.72 0)
-      (effects (font (size 1.524 1.524)) hide)
-    )
-    (property "Value" "" (id 1) (at 146.05 167.64 0)
-      (effects (font (size 1.524 1.524)) hide)
-    )
-    (property "Footprint" "" (id 2) (at 146.05 170.18 0)
-      (effects (font (size 1.524 1.524)) hide)
-    )
-    (property "Datasheet" "" (id 3) (at 146.05 170.18 0)
+  (symbol (lib_id "artemisa:VCC") (at 139.7 41.91 0) (unit 1)
+    (in_bom yes) (on_board yes)
+    (property "Reference" "#PWR091" (id 0) (at 139.7 43.18 0)
+      (effects (font (size 1.524 1.524)) hide)
+    )
+    (property "Value" "VCC" (id 1) (at 139.7 35.56 0)
+      (effects (font (size 1.524 1.524)) hide)
+    )
+    (property "Footprint" "" (id 2) (at 139.7 41.91 0)
+      (effects (font (size 1.524 1.524)) hide)
+    )
+    (property "Datasheet" "" (id 3) (at 139.7 41.91 0)
+      (effects (font (size 1.524 1.524)) hide)
+    )
+    (pin "1")
+  )
+  (symbol (lib_id "artemisa:GND") (at 139.7 102.87 0) (unit 1)
+    (in_bom yes) (on_board yes)
+    (property "Reference" "#PWR092" (id 0) (at 139.7 105.41 0)
+      (effects (font (size 1.524 1.524)) hide)
+    )
+    (property "Value" "GND" (id 1) (at 139.7 100.33 0)
+      (effects (font (size 1.524 1.524)) hide)
+    )
+    (property "Footprint" "" (id 2) (at 139.7 102.87 0)
+      (effects (font (size 1.524 1.524)) hide)
+    )
+    (property "Datasheet" "" (id 3) (at 139.7 102.87 0)
       (effects (font (size 1.524 1.524)) hide)
     )
     (pin "~")
   )
-  (symbol (lib_id "artemisa:VCC") (at 139.7 41.91 0) (unit 1)
-    (in_bom yes) (on_board yes)
-    (property "Reference" "#PWR060" (id 0) (at 139.7 43.18 0)
-      (effects (font (size 1.524 1.524)) hide)
-    )
-    (property "Value" "" (id 1) (at 139.7 35.56 0)
-      (effects (font (size 1.524 1.524)) hide)
-    )
-    (property "Footprint" "" (id 2) (at 139.7 41.91 0)
-      (effects (font (size 1.524 1.524)) hide)
-    )
-    (property "Datasheet" "" (id 3) (at 139.7 41.91 0)
-      (effects (font (size 1.524 1.524)) hide)
-    )
-    (pin "~")
-  )
-  (symbol (lib_id "artemisa:GND") (at 139.7 102.87 0) (unit 1)
-    (in_bom yes) (on_board yes)
-    (property "Reference" "#PWR063" (id 0) (at 139.7 105.41 0)
-      (effects (font (size 1.524 1.524)) hide)
-    )
-    (property "Value" "" (id 1) (at 139.7 100.33 0)
-      (effects (font (size 1.524 1.524)) hide)
-    )
-    (property "Footprint" "" (id 2) (at 139.7 102.87 0)
-      (effects (font (size 1.524 1.524)) hide)
-    )
-    (property "Datasheet" "" (id 3) (at 139.7 102.87 0)
-      (effects (font (size 1.524 1.524)) hide)
-    )
-    (pin "~")
-  )
   (symbol (lib_id "artemisa:Cap") (at 147.32 44.45 90) (unit 1)
     (in_bom yes) (on_board yes)
-    (property "Reference" "C?" (id 0) (at 146.05 43.18 90)
+    (property "Reference" "C33" (id 0) (at 146.05 43.18 90)
       (effects (font (size 1.27 1.27)) (justify left))
     )
-    (property "Value" "" (id 1) (at 154.94 43.18 90)
+    (property "Value" "100nF" (id 1) (at 154.94 43.18 90)
       (effects (font (size 1.27 1.27)) (justify left))
     )
-    (property "Footprint" "" (id 2) (at 147.32 44.45 0)
+    (property "Footprint" "artemisa:Disc_capacitor" (id 2) (at 147.32 44.45 0)
       (effects (font (size 1.27 1.27)) hide)
     )
@@
   (symbol (lib_id "artemisa:GND") (at 153.67 46.99 0) (unit 1)
     (in_bom yes) (on_board yes)
-    (property "Reference" "#PWR061" (id 0) (at 153.67 49.53 0)
-      (effects (font (size 1.524 1.524)) hide)
-    )
-    (property "Value" "" (id 1) (at 153.67 44.45 0)
-      (effects (font (size 1.524 1.524)) hide)
-    )
+    (property "Reference" "#PWR095" (id 0) (at 153.67 49.53 0)
+      (effects (font (size 1.524 1.524)) hide)
+    )
+    (property "Value" "GND" (id 1) (at 153.67 44.45 0)
+      (effects (font (size 1.524 1.524)) hide)
+    )
