File: slots.kicad_sch (KiCad schematic)
At the start: 6 parts

Commit message: Implement power transform circuit
Parts:
- C36: renamed from C?; value (none) -> 100nF; footprint (none) -> artemisa:Disc_capacitor
- J2: renamed from J3; value (none) -> MSX_Slot; footprint (none) -> artemisa:Slot_conn
- J3: renamed from J4; value (none) -> MSX_Slot; footprint (none) -> artemisa:Slot_conn
- J4: renamed from J5; value (none) -> GFX_Connector_Output; footprint (none) -> artemisa:GFX_conn
- RN3: value (none) -> 10K; footprint (none) -> artemisa:RN6
- U28: renamed from U18; value (none) -> 74HCT08; footprint (none) -> artemisa:DIP-14_300
Connections:
- net VCC: now also C36.1, J2.45 (Pin_45), J2.47 (Pin_47), J3.45 (Pin_45), J3.47 (Pin_47), J4.4 (~{SLTSL}), J4.45 (5V), J4.47 (5V), RN3.1, U28.14 (VCC)
